Commit message: added inertia values

File: src/arduinobot_description/urdf/arduinobot.urdf.xacro (robot description, xacro)
@@ -13,18 +13,14 @@
     <xacro:property name="effort" value="30.0" />
     <xacro:property name="velocity" value="10.0" />
-    <!-- Useful Macros -->
-    <xacro:macro name="default_inertial" params="mass">
-        <inertial>
-            <origin xyz="0 0 0" rpy="0 0 0"/>
-            <mass value="${mass}" />
-            <inertia ixx="1.0" ixy="0.0" ixz="0.0"
-                     iyy="1.0" iyz="0.0"
-                     izz="1.0" />
-        </inertial>
-    </xacro:macro>
     <!-- Links -->
     <link name="world"/>
     <link name="base_link">
-        <xacro:default_inertial mass="1.0"/>
+        <inertial>
+            <origin xyz="0.047813751 0.050114205 0.011410979" rpy="0 0 0"/>
+            <mass value="0.053288777" />
+            <inertia ixx="3.37E-05" ixy="3.35E-09" ixz="-4.41E-10"
+                     iyy="3.12E-05" iyz="9.25E-08"
+                     izz="5.65E-05" />
+        </inertial>
         <visual>
             <origin rpy="0 0 0" xyz="-0.5 -0.5 0"/>
@@ -41,5 +37,11 @@
     </link>
     <link name="base_plate">
-        <xacro:default_inertial mass="0.1"/>
+        <inertial>
+            <origin xyz="0.03745683 0.039132251 0.068646169" rpy="0 0 0"/>
+            <mass value="0.054531064" />
+            <inertia ixx="2.30E-05" ixy="-2.08E-06" ixz="1.93E-06"
+                     iyy="2.75E-05" iyz="-2.33E-06"
+                     izz="3.20E-05" />
+        </inertial>
         <visual>
             <origin rpy="0 0 0" xyz="-0.39 -0.39 -0.56"/>
@@ -56,5 +58,11 @@
     </link>
     <link name="forward_drive_arm">
-        <xacro:default_inertial mass="0.1"/>
+        <inertial>
+            <origin xyz="0.041356854 0.015301914 0.006504508" rpy="0 0 0"/>
+            <mass value="0.016329173" />
+            <inertia ixx="1.29E-06" ixy="-1.85E-07" ixz="-3.52E-07"
+                     iyy="1.17E-05" iyz="5.31E-09"
+                     izz="1.25E-05" />
+        </inertial>
         <visual>
             <origin rpy=" 0 -${PI / 2} ${PI / 2}" xyz="0.19 0.06 -0.08"/>
@@ -71,5 +79,11 @@
     </link>
     <link name="horizontal_arm">
-        <xacro:default_inertial mass="0.1"/>
+        <inertial>
+            <origin xyz="0.05942601 0.007996574 0.00404" rpy="0 0 0"/>
+            <mass value="0.01094525" />
+            <inertia ixx="2.38E-07" ixy="-1.58E-07" ixz="5.44E-14"
+                     iyy="1.49E-05" iyz="-4.00E-14"
+                     izz="1.50E-05" />
+        </inertial>
         <visual>
             <origin rpy="${PI / 2} 0 ${PI / 2}" xyz="-0.03 -0.4 -0.06"/>
@@ -86,5 +100,11 @@
     </link>
     <link name="claw_support">
-        <xacro:default_inertial mass="0.05"/>
+        <inertial>
+            <origin xyz="0.019393395 0.011560624 0.010132371" rpy="0 0 0"/>
+            <mass value="0.008336755" />
+            <inertia ixx="1.39E-06" ixy="5.05E-08" ixz="-4.60E-07"
+                     iyy="2.82E-06" iyz="-1.60E-07"
+                     izz="2.19E-06" />
+        </inertial>
         <visual>
             <origin rpy="0 0 ${PI / 2}" xyz="0 -0.05 -0.15"/>
@@ -101,5 +121,11 @@
     </link>
     <link name="gripper_right">
-        <xacro:default_inertial mass="0.01"/>
+        <inertial>
+            <origin xyz="0.029137181 0.008193029 0.002098195" rpy="0 0 0"/>
+            <mass value="0.001830792" />
+            <inertia ixx="2.98E-08" ixy="3.93E-08" ixz="-2.07E-08"
+                     iyy="5.41E-07" iyz="-4.79E-09"
+                     izz="5.60E-07" />
+        </inertial>
         <visual>
             <origin rpy="0 0 -${PI / 2}" xyz="-0.1 0.50 -0.1"/>
@@ -116,5 +142,11 @@
     </link>
     <link name="gripper_left">
-        <xacro:default_inertial mass="0.01"/>
+        <inertial>
+            <origin xyz="0.028124305 0.006099151 0.002138814" rpy="0 0 0"/>
+            <mass value="0.001736879" />
+            <inertia ixx="2.87E-08" ixy="-3.36E-08" ixz="-1.93E-08"
+                     iyy="5.03E-07" iyz="4.60E-09"
+                     izz="5.20E-07" />
+        </inertial>
         <visual>
             <origin rpy="0 0 -${PI / 2}" xyz="-0.04 0.50 -0.1"/>
